Commit message: Some basic interfacing is now possible in Gazebo!

File: little_pig_description/urdf/basic_geometry_pig.urdf.xacro (robot description, xacro)
@@ -62,14 +62,33 @@
         </link>
         <!-- The Joint -->
-        <joint name="${prefix}_ackerman_link_joint" type="revolute">
+        <joint name="base_link_${prefix}_ackerman_link" type="revolute">
             <axis xyz="0.0 0.0 1.0" rpy="0.0 0.0 0.0"/>
             <parent link="base_link"/>
             <child link="${prefix}_ackerman_link"/>
             <origin xyz="${length / 2.5} ${((ackerman_joint_width/2) + (width/2)) * reflect} -${(height / 2.25) + (ackerman_joint_diameter / 2)}" rpy="0.0 0.0 0.0"/>
-            <limit lower="-0.5" upper="0.5" effort="0.0" velocity="0.0"/>
+            <limit lower="-0.5" upper="0.5" effort="1.0" velocity="0.1"/>
         </joint>
+        <!-- Gazebo Interface -->
+        <gazebo reference="${prefix}_ackerman_link">
+            <mu1 value="200.0"/>
+            <mu2 value="100.0"/>
+            <kp value="10000000.0" />
+            <kd value="1.0" />
+            <material>Gazebo/Blue</material>
+        </gazebo>
+        <!-- The Transmission -->
+        <transmission name="base_link_${prefix}_ackerman_link_trans">
+            <type>transmission_interface/SimpleTransmission</type>
+            <joint name="base_link_${prefix}_ackerman_link">
+                <hardwareInterface>EffortJointInterface</hardwareInterface>
+            </joint>
+            <actuator name="base_link_${prefix}_ackerman_link_motor">
+                <hardwareInterface>EffortJointInterface</hardwareInterface>
+                <mechanicalReduction>1</mechanicalReduction>
+            </actuator>
+        </transmission>
     </xacro:macro>
     <!-- Front Wheel Macro -->
-    <xacro:macro name="front_wheel" params="suffix reflect">
+    <xacro:macro name="front_wheel" params="prefix suffix reflect">
         <!-- The Link -->
         <link name="front_${suffix}_wheel">
@@ -94,7 +113,7 @@
         </link>
         <!-- The Joint -->
-        <joint name="ackerman_steering_to_front_${suffix}_wheel" type="continuous">
-            <axis xyz="0.0 0.1 0.0"/>
-            <parent link="${suffix}_ackerman_link"/>
+        <joint name="${prefix}_ackerman_link_front_${suffix}_wheel" type="continuous">
+            <axis xyz="0.0 1.0 0.0"/>
+            <parent link="${prefix}_ackerman_link"/>
             <child link="front_${suffix}_wheel"/>
             <origin xyz="0.0 0.0 0.0" rpy="0.0 0.0 0.0"/>
@@ -109,10 +128,10 @@
         </gazebo>
         <!-- The Transmission -->
-        <transmission name="front_${suffix}_wheel_trans">
+        <transmission name="${prefix}_ackerman_link_front_${suffix}_wheel_trans">
             <type>transmission_interface/SimpleTransmission</type>
-            <joint name="ackerman_steering_to_front_${suffix}_wheel">
+            <joint name="${prefix}_ackerman_link_front_${suffix}_wheel">
                 <hardwareInterface>EffortJointInterface</hardwareInterface>
             </joint>
-            <actuator name="front_${suffix}_wheel_motor">
+            <actuator name="${prefix}_ackerman_link_front_${suffix}_wheel_motor">
                 <hardwareInterface>EffortJointInterface</hardwareInterface>
                 <mechanicalReduction>1</mechanicalReduction>
@@ -155,6 +174,6 @@
     <xacro:ackerman_steering prefix="right" reflect="-1" />
     <!-- Call the front wheels in left/right -->
-    <xacro:front_wheel suffix="left" reflect="1" />
-    <xacro:front_wheel suffix="right" reflect="-1" />
+    <xacro:front_wheel prefix="left" suffix="left" reflect="1" />
+    <xacro:front_wheel prefix="right" suffix="right" reflect="-1" />
     <!-- Call the rear wheels in left/right-->
     <xacro:rear_wheel suffix="left" reflect="1" />

Commit message: Getting very

File: little_pig_description/urdf/basic_geometry_pig.urdf.xacro (robot description, xacro)
@@ -39,7 +39,15 @@
             <origin xyz="0.0 0.0 0.0" rpy="0.0 0.0 0.0"/>
             <mass value="49.8952"/>
-            <inertia ixx="11.48" ixy="10.52" ixz="1.737" iyy="1.737" iyz="11.48" izz="10.52"/>
+            <inertia ixx="11.48" ixy="0.0" ixz="0.0" iyy="1.737" iyz="0.0" izz="10.52"/>
         </inertial>
     </link>
+    <!-- Gazebo Interface -->
+    <gazebo reference="base_link">
+        <mu1 value="0.0"/>
+        <mu2 value="0.0"/>
+        <kp value="10000000.0" />
+        <kd value="1.0" />
+        <material>Gazebo/Blue</material>
+    </gazebo>
     <!-- Ackerman Steering Macro -->
     <xacro:macro name="ackerman_steering" params="prefix reflect">
@@ -67,13 +75,14 @@
             <child link="${prefix}_ackerman_link"/>
             <origin xyz="${length / 2.5} ${((ackerman_joint_width/2) + (width/2)) * reflect} -${(height / 2.25) + (ackerman_joint_diameter / 2)}" rpy="0.0 0.0 0.0"/>
-            <limit lower="-0.5" upper="0.5" effort="1.0" velocity="0.1"/>
+            <limit lower="-0.5" upper="0.5" effort="20.0" velocity="2.0"/>
         </joint>
         <!-- Gazebo Interface -->
         <gazebo reference="${prefix}_ackerman_link">
-            <mu1 value="200.0"/>
-            <mu2 value="100.0"/>
+            <mu1 value="1.0"/>
+            <mu2 value="1.0"/>
             <kp value="10000000.0" />
             <kd value="1.0" />
-            <material>Gazebo/Blue</material>
+            <fdir1 value="1 0 0"/>
+            <material>Gazebo/Black</material>
         </gazebo>
         <!-- The Transmission -->
@@ -118,11 +127,13 @@
             <child link="front_${suffix}_wheel"/>
             <origin xyz="0.0 0.0 0.0" rpy="0.0 0.0 0.0"/>
+            <limit lower="0.0" upper="0.0" effort="10" velocity="100"/>
         </joint>
         <!-- Gazebo Interface -->
         <gazebo reference="front_${suffix}_wheel">
-            <mu1 value="200.0"/>
-            <mu2 value="100.0"/>
+            <mu1 value="1.0"/>
+            <mu2 value="1.0"/>
             <kp value="10000000.0" />
             <kd value="1.0" />
+            <fdir1 value="0 0 1"/>
             <material>Gazebo/Black</material>
         </gazebo>
@@ -168,5 +179,26 @@
             <child link="rear_${suffix}_wheel"/>
             <origin xyz="-${length / 2.5} ${(width /2) * reflect} -${(height / 5) + (rear_wheel_diameter / 2)}" rpy="0.0 0.0 0.0"/>
+            <limit lower="0.0" upper="0.0" effort="10" velocity="100"/>
         </joint>
+        <!-- Gazebo Interface -->
+        <gazebo reference="rear_${suffix}_wheel">
+            <mu1 value="1.0"/>
+            <mu2 value="1.0"/>
+            <kp value="10000000.0" />
+            <kd value="1.0" />
+            <fdir1 value="1 0 0"/>
+            <material>Gazebo/Black</material>
+        </gazebo>
+        <!-- The Transmission -->
+        <transmission name="base_to_rear_${suffix}_wheel_trans">
+            <type>transmission_interface/SimpleTransmission</type>
+            <joint name="base_to_rear_${suffix}_wheel">
+                <hardwareInterface>EffortJointInterface</hardwareInterface>
+            </joint>
+            <actuator name="base_to_rear_${suffix}_wheel_motor">
+                <hardwareInterface>EffortJointInterface</hardwareInterface>
+                <mechanicalReduction>1</mechanicalReduction>
+            </actuator>
+        </transmission>
     </xacro:macro>
     <!-- Call the ackermans in for left/right -->

Commit message: Updating Basic Geomtry Pig

File: little_pig_description/urdf/basic_geometry_pig.urdf.xacro (robot description, xacro)
@@ -4,4 +4,9 @@
     <!-- Standard Params -->
     <xacro:property name="pi" value="3.1415" />
+    <!-- Degree-to-radian conversions -->
+    <xacro:property name="degrees_45" value="0.785398163"/>
+    <xacro:property name="degrees_90" value="1.57079633"/>
+    <xacro:property name="degrees_180" value="3.14159265"/>
+    <!-- Inertia Generator -->
     <xacro:macro name="default_inertial" params="mass">
         <inertial>
@@ -10,4 +15,17 @@
         </inertial>
     </xacro:macro>
+    <!-- axle eff limit = 2 * stall_torque
+       as a function of the max gradient (15%) with overall max payload (600Kg) * wheel_radius
+       (calculating this way, it should be divided by 2 if 2 motors are used)
+       axle_eff_limit = 204.95 / 2 N m = ~102.5 -->
+    <!-- xacro:property name="axle_eff_limit" value="102.5"/ -->
+    <xacro:property name="axle_eff_limit" value="204.95"/>
+    <!-- max_speed = 33 Km/h = 9.17 m/s
+       axle_vel_limit = (2 * pi) * (max_speed / (pi * tire_dia)) =  39.02 rad/s -->
+    <xacro:property name="axle_vel_limit" value="39.02"/>
+    <!-- Servo_stall_torque of the direction axis in Nm. servo_no_load_speed is
+       measured in rad/s. -->
+    <xacro:property name="servo_stall_torque" value="50"/>
+    <xacro:property name="servo_no_load_speed" value="25"/>
     <!-- Basic Geometry of Body -->
     <xacro:property name="width" value="0.680618" />
@@ -44,8 +62,4 @@
     <!-- Gazebo Interface -->
     <gazebo reference="base_link">
-        <mu1 value="0.0"/>
-        <mu2 value="0.0"/>
-        <kp value="10000000.0" />
-        <kd value="1.0" />
         <material>Gazebo/Blue</material>
     </gazebo>
@@ -75,5 +89,5 @@
             <child link="${prefix}_ackerman_link"/>
             <origin xyz="${length / 2.5} ${((ackerman_joint_width/2) + (width/2)) * reflect} -${(height / 2.25) + (ackerman_joint_diameter / 2)}" rpy="0.0 0.0 0.0"/>
-            <limit lower="-0.5" upper="0.5" effort="20.0" velocity="2.0"/>
+            <limit lower="${-degrees_45}" upper="${degrees_45}" effort="${servo_stall_torque}" velocity="${servo_no_load_speed}"/>
         </joint>
         <!-- Gazebo Interface -->
@@ -90,8 +104,8 @@
             <type>transmission_interface/SimpleTransmission</type>
             <joint name="base_link_${prefix}_ackerman_link">
-                <hardwareInterface>EffortJointInterface</hardwareInterface>
+                <hardwareInterface>hardware_interface/EffortJointInterface</hardwareInterface>
             </joint>
             <actuator name="base_link_${prefix}_ackerman_link_motor">
-                <hardwareInterface>EffortJointInterface</hardwareInterface>
+                <hardwareInterface>hardware_interface/EffortJointInterface</hardwareInterface>
                 <mechanicalReduction>1</mechanicalReduction>
             </actuator>
@@ -142,8 +156,8 @@
             <type>transmission_interface/SimpleTransmission</type>
             <joint name="${prefix}_ackerman_link_front_${suffix}_wheel">
-                <hardwareInterface>EffortJointInterface</hardwareInterface>
+                <hardwareInterface>hardware_interface/VelocityJointInterface</hardwareInterface>
             </joint>
             <actuator name="${prefix}_ackerman_link_front_${suffix}_wheel_motor">
-                <hardwareInterface>EffortJointInterface</hardwareInterface>
+                <hardwareInterface>hardware_interface/VelocityJointInterface</hardwareInterface>
                 <mechanicalReduction>1</mechanicalReduction>
             </actuator>
@@ -194,8 +208,8 @@
             <type>transmission_interface/SimpleTransmission</type>
             <joint name="base_to_rear_${suffix}_wheel">
-                <hardwareInterface>EffortJointInterface</hardwareInterface>
+                <hardwareInterface>hardware_interface/VelocityJointInterface</hardwareInterface>
             </joint>
             <actuator name="base_to_rear_${suffix}_wheel_motor">
-                <hardwareInterface>EffortJointInterface</hardwareInterface>
+                <hardwareInterface>hardware_interface/VelocityJointInterface</hardwareInterface>
                 <mechanicalReduction>1</mechanicalReduction>
             </actuator>

Commit message: FUCK ROS!!!!!!!!!!!!!!!!!!!!!!!!!!!!!!!!!!!!!!!!!

File: little_pig_description/urdf/basic_geometry_pig.urdf.xacro (robot description, xacro)
@@ -15,17 +15,10 @@
         </inertial>
     </xacro:macro>
-    <!-- axle eff limit = 2 * stall_torque
-       as a function of the max gradient (15%) with overall max payload (600Kg) * wheel_radius
-       (calculating this way, it should be divided by 2 if 2 motors are used)
-       axle_eff_limit = 204.95 / 2 N m = ~102.5 -->
-    <!-- xacro:property name="axle_eff_limit" value="102.5"/ -->
-    <xacro:property name="axle_eff_limit" value="204.95"/>
-    <!-- max_speed = 33 Km/h = 9.17 m/s
-       axle_vel_limit = (2 * pi) * (max_speed / (pi * tire_dia)) =  39.02 rad/s -->
+    <xacro:property name="axle_eff_limit" value="100"/>
     <xacro:property name="axle_vel_limit" value="39.02"/>
     <!-- Servo_stall_torque of the direction axis in Nm. servo_no_load_speed is
        measured in rad/s. -->
-    <xacro:property name="servo_stall_torque" value="50"/>
-    <xacro:property name="servo_no_load_speed" value="25"/>
+    <xacro:property name="servo_stall_torque" value="100"/>
+    <xacro:property name="servo_no_load_speed" value="100"/>
     <!-- Basic Geometry of Body -->
     <xacro:property name="width" value="0.680618" />
@@ -141,5 +134,5 @@
             <child link="front_${suffix}_wheel"/>
             <origin xyz="0.0 0.0 0.0" rpy="0.0 0.0 0.0"/>
-            <limit lower="0.0" upper="0.0" effort="10" velocity="100"/>
+            <limit effort="${axle_eff_limit}" velocity="${axle_vel_limit}"/>
         </joint>
         <!-- Gazebo Interface -->
@@ -193,13 +186,12 @@
             <child link="rear_${suffix}_wheel"/>
             <origin xyz="-${length / 2.5} ${(width /2) * reflect} -${(height / 5) + (rear_wheel_diameter / 2)}" rpy="0.0 0.0 0.0"/>
-            <limit lower="0.0" upper="0.0" effort="10" velocity="100"/>
         </joint>
         <!-- Gazebo Interface -->
         <gazebo reference="rear_${suffix}_wheel">
-            <mu1 value="1.0"/>
+            <!-- <mu1 value="1.0"/>
             <mu2 value="1.0"/>
             <kp value="10000000.0" />
             <kd value="1.0" />
-            <fdir1 value="1 0 0"/>
+            <fdir1 value="1 0 0"/> -->
             <material>Gazebo/Black</material>
         </gazebo>
