Commit message: Updated Inertias on the Basic Frame Pig

File: little_pig_description/urdf/basic_frame_pig.urdf.xacro (robot description, xacro)
@@ -1,11 +1,23 @@
 <?xml version="1.0"?>
-<robot name="basic_frame_pig">
+<robot name="basic_frame_pig"
+    xmlns:xacro="http://www.ros.org/wiki/xacro">
+    <!-- Null inertial element. This is needed to make the model work with
+       Gazebo. -->
+    <xacro:macro name="null_inertial">
+        <inertial>
+            <mass value="0.001"/>
+            <inertia ixx="0.001" ixy="0" ixz="0" iyy="0.001" iyz="0" izz="0.001"/>
+        </inertial>
+    </xacro:macro>
     <!-- Base Link / Tube Chasis-->
     <link name="base_link">
-        <inertial>
+        <!-- Load Gazebo Inertial -->
+        <xacro:null_inertial/>
+        <!-- These Inertias are not suitable with Gazebo -->
+        <!-- <inertial>
             <origin rpy="0 0 0" xyz="-0.005632841369081588 0.2917022138225285 -0.004107516953549188"/>
             <mass value="61.719091558990335"/>
             <inertia ixx="23.451972" ixy="-0.091403" ixz="-0.110297" iyy="6.432858" iyz="1.415813" izz="26.484945"/>
-        </inertial>
+        </inertial> -->
         <visual>
             <origin rpy="0 0 0" xyz="0 0 0"/>
@@ -26,9 +38,12 @@
     <!-- Left Steering Knuckle -->
     <link name="left_steering_knuckle">
-        <inertial>
+        <!-- Load Gazebo Inertial -->
+        <xacro:null_inertial/>
+        <!-- These Inertias are not suitable with Gazebo -->
+        <!-- <inertial>
             <origin rpy="0 0 0" xyz="0.04626374762862234 0.005213062909487198 0.06475119586205944"/>
             <mass value="2.3221244569381487"/>
             <inertia ixx="0.004736" ixy="0.000171" ixz="6.1e-05" iyy="0.003675" iyz="6e-06" izz="0.003101"/>
-        </inertial>
+        </inertial> -->
         <visual>
             <origin rpy="0 0 0" xyz="-0.447222 0.622377 0.163596"/>
@@ -68,9 +83,12 @@
     <!-- Front Left Wheel Hub -->
     <link name="front_left_wheel_hub">
-        <inertial>
+        <!-- Load Gazebo Inertial -->
+        <xacro:null_inertial/>
+        <!-- These Inertias are not suitable with Gazebo -->
+        <!-- <inertial>
             <origin rpy="0 0 0" xyz="0.027160820485626624 1.743857634961543e-07 0.0010195880848413164"/>
             <mass value="1.118795265201953"/>
             <inertia ixx="0.001287" ixy="-0.0" ixz="1.1e-05" iyy="0.000986" iyz="0.0" izz="0.000987"/>
-        </inertial>
+        </inertial> -->
         <visual>
             <origin rpy="0 0 0" xyz="-0.526843 0.622377 0.097593"/>
@@ -109,9 +127,12 @@
     <!-- Front Left Wheel -->
     <link name="front_left_wheel">
-        <inertial>
+        <!-- Load Gazebo Inertial -->
+        <xacro:null_inertial/>
+        <!-- These Inertias are not suitable with Gazebo -->
+        <!-- <inertial>
             <origin rpy="0 0 0" xyz="0.0011488911139707625 2.510309293879409e-06 3.8079092190917985e-05"/>
             <mass value="77.98350831979032"/>
             <inertia ixx="4.69787" ixy="-9e-06" ixz="0.077554" iyy="2.63247" iyz="-3e-05" izz="2.635399"/>
-        </inertial>
+        </inertial> -->
         <visual>
             <origin rpy="0 0 0" xyz="-0.563887 0.622377 0.096202"/>
@@ -149,9 +170,12 @@
     <!-- Right Steering Knuckle -->
     <link name="right_steering_knuckle">
-        <inertial>
+        <!-- Load Gazebo Inertial -->
+        <xacro:null_inertial/>
+        <!-- These Inertias are not suitable with Gazebo -->
+        <!-- <inertial>
             <origin rpy="0 0 0" xyz="-0.04602703865184993 0.00521305901325253 0.06491864444227143"/>
             <mass value="2.322126893861874"/>
             <inertia ixx="0.004736" ixy="-0.000171" ixz="-6.7e-05" iyy="0.003675" iyz="7e-06" izz="0.003102"/>
-        </inertial>
+        </inertial> -->
         <visual>
             <origin rpy="0 0 0" xyz="0.457954 0.622377 0.162568"/>
@@ -191,9 +215,12 @@
     <!-- Front Right Wheel Hub -->
     <link name="front_right_wheel_hub">
-        <inertial>
+        <!-- Load Gazebo Inertial -->
+        <xacro:null_inertial/>
+        <!-- These Inertias are not suitable with Gazebo -->
+        <!-- <inertial>
             <origin rpy="0 0 0" xyz="-0.03807755669639501 2.229040352297318e-07 0.0015684173363760129"/>
             <mass value="1.1187951842239643"/>
             <inertia ixx="0.001286" ixy="0.0" ixz="-1.2e-05" iyy="0.000986" iyz="-0.0" izz="0.000987"/>
-        </inertial>
+        </inertial> -->
         <visual>
             <origin rpy="0 0 0" xyz="0.526428 0.622377 0.096724"/>
@@ -232,9 +259,12 @@
     <!-- Front Right Wheel -->
     <link name="front_right_wheel">
-        <inertial>
+        <!-- Load Gazebo Inertial -->
+        <xacro:null_inertial/>
+        <!-- These Inertias are not suitable with Gazebo -->
+        <!-- <inertial>
             <origin rpy="0 0 0" xyz="-0.001292276290758898 2.291232137796584e-06 5.7530997634336334e-05"/>
             <mass value="77.98348447888712"/>
             <inertia ixx="4.697279" ixy="1.1e-05" ixz="-0.085043" iyy="2.632396" iyz="2.9e-05" izz="2.635914"/>
-        </inertial>
+        </inertial> -->
         <visual>
             <origin rpy="0 0 0" xyz="0.574387 0.622377 0.094748"/>
@@ -272,4 +302,7 @@
     <!-- Rear Left Wheel Hub -->
     <link name="rear_left_hub">
+        <!-- Load Gazebo Inertial -->
+        <xacro:null_inertial/>
+        <!-- These Inertias are not suitable with Gazebo -->
         <inertial>
             <origin rpy="0 0 0" xyz="0.027291669153874487 1.9676759810405287e-07 -0.0001474093893083922"/>
@@ -313,9 +346,12 @@
     <!-- Rear Left Wheel -->
     <link name="rear_left_wheel">
-        <inertial>
+        <!-- Load Gazebo Inertial -->
+        <xacro:null_inertial/>
+        <!-- These Inertias are not suitable with Gazebo -->
+        <!-- <inertial>
             <origin rpy="0 0 0" xyz="-0.024998897547842458 3.7973710019789664e-06 0.0001368244068725294"/>
             <mass value="88.28370410127773"/>
             <inertia ixx="5.402188" ixy="-3e-05" ixz="-0.011694" iyy="3.237533" iyz="2.6e-05" izz="3.237567"/>
-        </inertial>
+        </inertial> -->
         <visual>
             <origin rpy="0 0 0" xyz="-0.584846 -0.788123 0.103034"/>
@@ -353,9 +389,12 @@
     <!-- Rear Right Wheel Hub -->
     <link name="rear_right_hub">
-        <inertial>
+        <!-- Load Gazebo Inertial -->
+        <xacro:null_inertial/>
+        <!-- These Inertias are not suitable with Gazebo -->
+        <!-- <inertial>
             <origin rpy="0 0 0" xyz="-0.027291096145922622 2.0521091637082378e-07 3.286601153970614e-05"/>
             <mass value="1.1187959967121328"/>
             <inertia ixx="0.001287" ixy="-0.0" ixz="-0.0" iyy="0.000986" iyz="-0.0" izz="0.000986"/>
-        </inertial>
+        </inertial> -->
         <visual>
             <origin rpy="0 0 0" xyz="0.547263 -0.788123 0.13233"/>
@@ -394,9 +433,12 @@
     <!-- Rear Right Wheel -->
     <link name="rear_right_wheel">
-        <inertial>
+        <!-- Load Gazebo Inertial -->
+        <xacro:null_inertial/>
+        <!-- These Inertias are not suitable with Gazebo -->
+        <!-- <inertial>
             <origin rpy="0 0 0" xyz="0.022815265177914767 2.0103108817615123e-06 -2.4107454217187074e-05"/>
             <mass value="88.28370095669479"/>
             <inertia ixx="5.402246" ixy="1.2e-05" ixz="-0.002585" iyy="3.234966" iyz="2.6e-05" izz="3.235"/>
-        </inertial>
+        </inertial> -->
         <visual>
             <origin rpy="0 0 0" xyz="0.584444 -0.788123 0.132285"/>
