Commit message: Making Some Changes to Basic Frame Pig

File: little_pig_description/urdf/basic_frame_pig.urdf.xacro (robot description, xacro)
@@ -2,4 +2,23 @@
 <robot name="basic_frame_pig"
     xmlns:xacro="http://www.ros.org/wiki/xacro">
+    <!-- Degree-to-radian conversions -->
+    <xacro:property name="degrees_45" value="0.785398163"/>
+    <xacro:property name="degrees_90" value="1.57079633"/>
+    <xacro:property name="degrees_180" value="3.14159265"/>
+    <!-- Servo_stall_torque of the direction axis in Nm. servo_no_load_speed is
+       measured in rad/s. -->
+    <xacro:property name="servo_stall_torque" value="50"/>
+    <xacro:property name="servo_no_load_speed" value="25"/>
+    <!-- axle eff limit = 2 * stall_torque
+       as a function of the max gradient (15%) with overall max payload (600Kg) * wheel_radius
+       (calculating this way, it should be divided by 2 if 2 motors are used)
+       axle_eff_limit = 204.95 / 2 N m = ~102.5 -->
+    <!-- xacro:property name="axle_eff_limit" value="102.5"/ -->
+    <xacro:property name="axle_eff_limit" value="204.95"/>
+    <!-- max_speed = 33 Km/h = 9.17 m/s
+       axle_vel_limit = (2 * pi) * (max_speed / (pi * tire_dia)) =  39.02 rad/s -->
+    <xacro:property name="axle_vel_limit" value="39.02"/>
+    <xacro:property name="wheel_joint_damping" value="0.2" />
+    <xacro:property name="wheel_joint_friction" value="0.7" />
     <!-- Null inertial element. This is needed to make the model work with
        Gazebo. -->
@@ -10,4 +29,48 @@
         </inertial>
     </xacro:macro>
+    <!-- Gazebo Interface -->
+    <gazebo reference="base_link">
+        <material>Gazebo/Grey</material>
+    </gazebo>
+    <!-- Gazebo Interface -->
+    <gazebo reference="left_steering_knuckle">
+        <material>Gazebo/Red</material>
+    </gazebo>
+    <!-- Gazebo Interface -->
+    <gazebo reference="front_left_wheel_hub">
+        <material>Gazebo/Blue</material>
+    </gazebo>
+    <!-- Gazebo Interface -->
+    <gazebo reference="front_left_wheel">
+        <material>Gazebo/Black</material>
+    </gazebo>
+    <!-- Gazebo Interface -->
+    <gazebo reference="right_steering_knuckle">
+        <material>Gazebo/Red</material>
+    </gazebo>
+    <!-- Gazebo Interface -->
+    <gazebo reference="front_right_wheel_hub">
+        <material>Gazebo/Blue</material>
+    </gazebo>
+    <!-- Gazebo Interface -->
+    <gazebo reference="front_Right_wheel">
+        <material>Gazebo/Black</material>
+    </gazebo>
+    <!-- Gazebo Interface -->
+    <gazebo reference="rear_left_hub">
+        <material>Gazebo/Blue</material>
+    </gazebo>
+    <!-- Gazebo Interface -->
+    <gazebo reference="rear_left_wheel">
+        <material>Gazebo/Black</material>
+    </gazebo>
+    <!-- Gazebo Interface -->
+    <gazebo reference="rear_right_hub">
+        <material>Gazebo/Blue</material>
+    </gazebo>
+    <!-- Gazebo Interface -->
+    <gazebo reference="rear_Right_wheel">
+        <material>Gazebo/Black</material>
+    </gazebo>
     <!-- Base Link / Tube Chasis-->
     <link name="base_link">
@@ -23,5 +86,5 @@
             <origin rpy="0 0 0" xyz="0 0 0"/>
             <geometry>
-                <mesh filename="package://little_pig_atv/urdf/bin_stl/base_link_m-binary.stl"/>
+                <mesh filename="package://little_pig_description/urdf/bin_stl/base_link_m-binary.stl"/>
             </geometry>
             <material name="silver">
@@ -32,5 +95,5 @@
             <origin rpy="0 0 0" xyz="0 0 0"/>
             <geometry>
-                <mesh filename="package://little_pig_atv/urdf/bin_stl/base_link_m-binary.stl"/>
+                <mesh filename="package://little_pig_description/urdf/bin_stl/base_link_m-binary.stl"/>
             </geometry>
         </collision>
@@ -49,5 +112,5 @@
             <origin rpy="0 0 0" xyz="-0.447222 0.622377 0.163596"/>
             <geometry>
-                <mesh filename="package://little_pig_atv/urdf/bin_stl/left_steering_knuckle_m-binary.stl"/>
+                <mesh filename="package://little_pig_description/urdf/bin_stl/left_steering_knuckle_m-binary.stl"/>
             </geometry>
             <material name="silver">
@@ -58,5 +121,5 @@
             <origin rpy="0 0 0" xyz="-0.447222 0.622377 0.163596"/>
             <geometry>
-                <mesh filename="package://little_pig_atv/urdf/bin_stl/left_steering_knuckle_m-binary.stl"/>
+                <mesh filename="package://little_pig_description/urdf/bin_stl/left_steering_knuckle_m-binary.stl"/>
             </geometry>
         </collision>
@@ -68,5 +131,5 @@
         <child link="left_steering_knuckle"/>
         <axis xyz="-0.000375 -0.0 0.009993"/>
-        <limit lower="-0.5" upper="0.5" effort="1.0" velocity="1.0"/>
+        <limit lower="${-degrees_45}" upper="${degrees_45}" effort="${servo_stall_torque}" velocity="${servo_no_load_speed}"/>
     </joint>
     <!-- Base Link - Left Steering Knuckle Transmission -->
@@ -74,8 +137,8 @@
         <type>transmission_interface/SimpleTransmission</type>
         <joint name="base_link_to_left_steering_knuckle">
-            <hardwareInterface>PositionJointInterface</hardwareInterface>
+            <hardwareInterface>hardware_interface/EffortJointInterface</hardwareInterface>
         </joint>
         <actuator name="base_link_to_left_steering_knuckle_actr">
-            <hardwareInterface>PositionJointInterface</hardwareInterface>
+            <hardwareInterface>hardware_interface/EffortJointInterface</hardwareInterface>
             <mechanicalReduction>1</mechanicalReduction>
         </actuator>
@@ -94,5 +157,5 @@
             <origin rpy="0 0 0" xyz="-0.526843 0.622377 0.097593"/>
             <geometry>
-                <mesh filename="package://little_pig_atv/urdf/bin_stl/front_left_wheel_hub_m-binary.stl"/>
+                <mesh filename="package://little_pig_description/urdf/bin_stl/front_left_wheel_hub_m-binary.stl"/>
             </geometry>
             <material name="silver">
@@ -103,5 +166,5 @@
             <origin rpy="0 0 0" xyz="-0.526843 0.622377 0.097593"/>
             <geometry>
-                <mesh filename="package://little_pig_atv/urdf/bin_stl/front_left_wheel_hub_m-binary.stl"/>
+                <mesh filename="package://little_pig_description/urdf/bin_stl/front_left_wheel_hub_m-binary.stl"/>
             </geometry>
         </collision>
@@ -113,4 +176,5 @@
         <child link="front_left_wheel_hub"/>
         <axis xyz="-0.009993 -0.0 -0.000375"/>
+        <limit effort="${axle_eff_limit}" velocity="${axle_vel_limit}"/>
     </joint>
     <!-- Front Left Steering Knuckle to Front Left Wheel Hub Transmission -->
@@ -118,8 +182,8 @@
         <type>transmission_interface/SimpleTransmission</type>
         <joint name="front_left_steering_knuckle_front_left_wheel_hub">
-            <hardwareInterface>EffortJointInterface</hardwareInterface>
+            <hardwareInterface>hardware_interface/VelocityJointInterface</hardwareInterface>
         </joint>
         <actuator name="front_left_steering_knuckle_front_left_wheel_hub_actr">
-            <hardwareInterface>EffortJointInterface</hardwareInterface>
+            <hardwareInterface>hardware_interface/VelocityJointInterface</hardwareInterface>
             <mechanicalReduction>1</mechanicalReduction>
         </actuator>
@@ -138,5 +202,5 @@
             <origin rpy="0 0 0" xyz="-0.563887 0.622377 0.096202"/>
             <geometry>
-                <mesh filename="package://little_pig_atv/urdf/bin_stl/front_left_wheel_m-binary.stl"/>
+                <mesh filename="package://little_pig_description/urdf/bin_stl/front_left_wheel_m-binary.stl"/>
             </geometry>
             <material name="silver">
@@ -147,5 +211,5 @@
             <origin rpy="0 0 0" xyz="-0.563887 0.622377 0.096202"/>
             <geometry>
-                <mesh filename="package://little_pig_atv/urdf/bin_stl/front_left_wheel_m-binary.stl"/>
+                <mesh filename="package://little_pig_description/urdf/bin_stl/front_left_wheel_m-binary.stl"/>
             </geometry>
         </collision>
@@ -158,5 +222,5 @@
     </joint>
     <!-- Front Left Wheel Hub to Front Left Wheel Joint-->
-    <transmission name="front_left_wheel_hub_front_left_wheel_transmission">
+    <!-- <transmission name="front_left_wheel_hub_front_left_wheel_transmission">
         <type>transmission_interface/SimpleTransmission</type>
         <joint name="front_left_wheel_hub_front_left_wheel">
@@ -167,5 +231,5 @@
             <mechanicalReduction>1</mechanicalReduction>
         </actuator>
-    </transmission>
+    </transmission> -->
     <!-- Right Steering Knuckle -->
     <link name="right_steering_knuckle">
@@ -181,5 +245,5 @@
             <origin rpy="0 0 0" xyz="0.457954 0.622377 0.162568"/>
             <geometry>
-                <mesh filename="package://little_pig_atv/urdf/bin_stl/right_steering_knuckle_m-binary.stl"/>
+                <mesh filename="package://little_pig_description/urdf/bin_stl/right_steering_knuckle_m-binary.stl"/>
             </geometry>
             <material name="silver">
@@ -190,5 +254,5 @@
             <origin rpy="0 0 0" xyz="0.457954 0.622377 0.162568"/>
             <geometry>
-                <mesh filename="package://little_pig_atv/urdf/bin_stl/right_steering_knuckle_m-binary.stl"/>
+                <mesh filename="package://little_pig_description/urdf/bin_stl/right_steering_knuckle_m-binary.stl"/>
             </geometry>
         </collision>
@@ -200,5 +264,5 @@
         <child link="right_steering_knuckle"/>
         <axis xyz="0.000412 -0.0 0.009992"/>
-        <limit lower="-0.5" upper="0.5" effort="1.0" velocity="1.0"/>
+        <limit lower="${-degrees_45}" upper="${degrees_45}" effort="${servo_stall_torque}" velocity="${servo_no_load_speed}"/>
     </joint>
     <!-- Base Link - Right Steering Knuckle Transmission -->
@@ -206,8 +270,8 @@
         <type>transmission_interface/SimpleTransmission</type>
         <joint name="base_link_to_right_steering_knuckle">
-            <hardwareInterface>PositionJointInterface</hardwareInterface>
+            <hardwareInterface>hardware_interface/EffortJointInterface</hardwareInterface>
         </joint>
         <actuator name="base_link_to_right_steering_knuckle_actr">
-            <hardwareInterface>PositionJointInterface</hardwareInterface>
+            <hardwareInterface>hardware_interface/EffortJointInterface</hardwareInterface>
             <mechanicalReduction>1</mechanicalReduction>
         </actuator>
@@ -226,5 +290,5 @@
             <origin rpy="0 0 0" xyz="0.526428 0.622377 0.096724"/>
             <geometry>
-                <mesh filename="package://little_pig_atv/urdf/bin_stl/front_right_wheel_hub_m-binary.stl"/>
+                <mesh filename="package://little_pig_description/urdf/bin_stl/front_right_wheel_hub_m-binary.stl"/>
             </geometry>
             <material name="silver">
@@ -235,5 +299,5 @@
             <origin rpy="0 0 0" xyz="0.526428 0.622377 0.096724"/>
             <geometry>
-                <mesh filename="package://little_pig_atv/urdf/bin_stl/front_right_wheel_hub_m-binary.stl"/>
+                <mesh filename="package://little_pig_description/urdf/bin_stl/front_right_wheel_hub_m-binary.stl"/>
             </geometry>
         </collision>
@@ -245,4 +309,5 @@
         <child link="front_right_wheel_hub"/>
         <axis xyz="0.009992 0.0 -0.000412"/>
+        <limit effort="${axle_eff_limit}" velocity="${axle_vel_limit}"/>
     </joint>
     <!-- Right Steering Knuckle - Front Right Wheel Hub Transmission -->
@@ -250,8 +315,8 @@
         <type>transmission_interface/SimpleTransmission</type>
         <joint name="right_steering_knuckle_front_right_hub">
-            <hardwareInterface>PositionJointInterface</hardwareInterface>
+            <hardwareInterface>hardware_interface/VelocityJointInterface</hardwareInterface>
         </joint>
         <actuator name="right_steering_knuckle_front_right_hub_actr">
-            <hardwareInterface>PositionJointInterface</hardwareInterface>
+            <hardwareInterface>hardware_interface/VelocityJointInterface</hardwareInterface>
             <mechanicalReduction>1</mechanicalReduction>
         </actuator>
@@ -270,5 +335,5 @@
             <origin rpy="0 0 0" xyz="0.574387 0.622377 0.094748"/>
             <geometry>
-                <mesh filename="package://little_pig_atv/urdf/bin_stl/front_right_wheel_m-binary.stl"/>
+                <mesh filename="package://little_pig_description/urdf/bin_stl/front_right_wheel_m-binary.stl"/>
             </geometry>
             <material name="silver">
@@ -279,5 +344,5 @@
             <origin rpy="0 0 0" xyz="0.574387 0.622377 0.094748"/>
             <geometry>
-                <mesh filename="package://little_pig_atv/urdf/bin_stl/front_right_wheel_m-binary.stl"/>
+                <mesh filename="package://little_pig_description/urdf/bin_stl/front_right_wheel_m-binary.stl"/>
             </geometry>
         </collision>
@@ -290,5 +355,5 @@
     </joint>
     <!-- Front Right Wheel Hub to Front Right Wheel Transmission -->
-    <transmission name="front_right_wheel_hub_front_right_wheel_transmission">
+    <!-- <transmission name="front_right_wheel_hub_front_right_wheel_transmission">
         <type>transmission_interface/SimpleTransmission</type>
         <joint name="front_right_wheel_hub_front_right_wheel">
@@ -299,5 +364,5 @@
             <mechanicalReduction>1</mechanicalReduction>
         </actuator>
-    </transmission>
+    </transmission> -->
     <!-- Rear Left Wheel Hub -->
     <link name="rear_left_hub">
@@ -313,5 +378,5 @@
             <origin rpy="0 0 0" xyz="-0.547664 -0.788123 0.102833"/>
             <geometry>
-                <mesh filename="package://little_pig_atv/urdf/bin_stl/rear_left_hub_m-binary.stl"/>
+                <mesh filename="package://little_pig_description/urdf/bin_stl/rear_left_hub_m-binary.stl"/>
             </geometry>
             <material name="silver">
@@ -322,5 +387,5 @@
             <origin rpy="0 0 0" xyz="-0.547664 -0.788123 0.102833"/>
             <geometry>
-                <mesh filename="package://little_pig_atv/urdf/bin_stl/rear_left_hub_m-binary.stl"/>
+                <mesh filename="package://little_pig_description/urdf/bin_stl/rear_left_hub_m-binary.stl"/>
             </geometry>
         </collision>
@@ -332,4 +397,5 @@
         <child link="rear_left_hub"/>
         <axis xyz="0.01 -0.0 -5.4e-05"/>
+        <limit effort="${axle_eff_limit}" velocity="${axle_vel_limit}"/>
     </joint>
     <!-- Base Link to Rear Left Wheel Hub Transmission -->
@@ -357,5 +423,5 @@
             <origin rpy="0 0 0" xyz="-0.584846 -0.788123 0.103034"/>
             <geometry>
-                <mesh filename="package://little_pig_atv/urdf/bin_stl/rear_left_wheel_m-binary.stl"/>
+                <mesh filename="package://little_pig_description/urdf/bin_stl/rear_left_wheel_m-binary.stl"/>
             </geometry>
             <material name="silver">
@@ -366,5 +432,5 @@
             <origin rpy="0 0 0" xyz="-0.584846 -0.788123 0.103034"/>
             <geometry>
-                <mesh filename="package://little_pig_atv/urdf/bin_stl/rear_left_wheel_m-binary.stl"/>
+                <mesh filename="package://little_pig_description/urdf/bin_stl/rear_left_wheel_m-binary.stl"/>
             </geometry>
         </collision>
@@ -400,5 +466,5 @@
             <origin rpy="0 0 0" xyz="0.547263 -0.788123 0.13233"/>
             <geometry>
-                <mesh filename="package://little_pig_atv/urdf/bin_stl/rear_right_hub_m-binary.stl"/>
+                <mesh filename="package://little_pig_description/urdf/bin_stl/rear_right_hub_m-binary.stl"/>
             </geometry>
             <material name="silver">
@@ -409,5 +475,5 @@
             <origin rpy="0 0 0" xyz="0.547263 -0.788123 0.13233"/>
             <geometry>
-                <mesh filename="package://little_pig_atv/urdf/bin_stl/rear_right_hub_m-binary.stl"/>
+                <mesh filename="package://little_pig_description/urdf/bin_stl/rear_right_hub_m-binary.stl"/>
             </geometry>
         </collision>
@@ -419,4 +485,5 @@
         <child link="rear_right_hub"/>
         <axis xyz="-0.01 0.0 1.2e-05"/>
+        <limit effort="${axle_eff_limit}" velocity="${axle_vel_limit}"/>
     </joint>
     <!-- Base Link to Rear Right Wheel Hub Transmission -->
@@ -444,5 +511,5 @@
             <origin rpy="0 0 0" xyz="0.584444 -0.788123 0.132285"/>
             <geometry>
-                <mesh filename="package://little_pig_atv/urdf/bin_stl/rear_right_wheel_m-binary.stl"/>
+                <mesh filename="package://little_pig_description/urdf/bin_stl/rear_right_wheel_m-binary.stl"/>
             </geometry>
             <material name="silver">
@@ -453,5 +520,5 @@
             <origin rpy="0 0 0" xyz="0.584444 -0.788123 0.132285"/>
             <geometry>
-                <mesh filename="package://little_pig_atv/urdf/bin_stl/rear_right_wheel_m-binary.stl"/>
+                <mesh filename="package://little_pig_description/urdf/bin_stl/rear_right_wheel_m-binary.stl"/>
             </geometry>
         </collision>

Commit message: I will never get this!!!!

File: little_pig_description/urdf/basic_frame_pig.urdf.xacro (robot description, xacro)
@@ -23,10 +23,10 @@
     <!-- Null inertial element. This is needed to make the model work with
        Gazebo. -->
-    <xacro:macro name="null_inertial">
+    <!-- <xacro:macro name="null_inertial">
         <inertial>
             <mass value="0.001"/>
             <inertia ixx="0.001" ixy="0" ixz="0" iyy="0.001" iyz="0" izz="0.001"/>
         </inertial>
-    </xacro:macro>
+    </xacro:macro> -->
     <!-- Gazebo Interface -->
     <gazebo reference="base_link">

Commit message: Got back wheels to move...

File: little_pig_description/urdf/basic_frame_pig.urdf.xacro (robot description, xacro)
@@ -397,8 +397,8 @@
         <child link="rear_left_hub"/>
         <axis xyz="0.01 -0.0 -5.4e-05"/>
-        <limit effort="${axle_eff_limit}" velocity="${axle_vel_limit}"/>
+        <!-- <limit effort="${axle_eff_limit}" velocity="${axle_vel_limit}"/> -->
     </joint>
     <!-- Base Link to Rear Left Wheel Hub Transmission -->
-    <transmission name="base_link_rear_left_wheel_hub_transmission">
+    <!-- <transmission name="base_link_rear_left_wheel_hub_transmission">
         <type>transmission_interface/SimpleTransmission</type>
         <joint name="base_link_rear_left_wheel_hub">
@@ -409,5 +409,5 @@
             <mechanicalReduction>1</mechanicalReduction>
         </actuator>
-    </transmission>
+    </transmission> -->
     <!-- Rear Left Wheel -->
     <link name="rear_left_wheel">
@@ -443,5 +443,5 @@
     </joint>
     <!-- Rear Left Wheel Hub to Rear Left Wheel Transmission -->
-    <transmission name="rear_left_wheel_hub_rear_left_wheel_transmission">
+    <!-- <transmission name="rear_left_wheel_hub_rear_left_wheel_transmission">
         <type>transmission_interface/SimpleTransmission</type>
         <joint name="rear_left_wheel_hub_rear_left_wheel">
@@ -452,5 +452,5 @@
             <mechanicalReduction>1</mechanicalReduction>
         </actuator>
-    </transmission>
+    </transmission> -->
     <!-- Rear Right Wheel Hub -->
     <link name="rear_right_hub">

File: little_pig_description/urdf/basic_geometry_pig.urdf.xacro (robot description, xacro)
@@ -197,5 +197,5 @@
         </gazebo>
         <!-- The Transmission -->
-        <transmission name="base_to_rear_${suffix}_wheel_trans">
+        <!-- <transmission name="base_to_rear_${suffix}_wheel_trans">
             <type>transmission_interface/SimpleTransmission</type>
             <joint name="base_to_rear_${suffix}_wheel">
@@ -206,5 +206,5 @@
                 <mechanicalReduction>1</mechanicalReduction>
             </actuator>
-        </transmission>
+        </transmission> -->
     </xacro:macro>
     <!-- Call the ackermans in for left/right -->
